File: pcb/windshield-wiper.sch (KiCad schematic (older format))
At the start: 22 parts

Commit message: KiCad files
Parts:
- removed K? (x3): SANYOU_SRD_Form_A, Relays_THT:Relay_SPDT_SANYOU_SRD_Series_Form_A, symbol SANYOU_SRD_Form_A
- removed SW?: SW_Rotary8, symbol SW_Rotary8
- added D1: LED, LEDs:LED_0805_HandSoldering, symbol LED
- added J2, J3: Screw_Terminal_01x03, TerminalBlock_Phoenix:TerminalBlock_Phoenix_MPT-2.54mm_3pol, symbol Screw_Terminal_01x03
- added J4: Screw_Terminal_01x02, TerminalBlock_Phoenix:TerminalBlock_Phoenix_MPT-2.54mm_2pol, symbol Screw_Terminal_01x02
- added J5: Screw_Terminal_01x05, TerminalBlock_Phoenix:TerminalBlock_Phoenix_MPT-2.54mm_5pol, symbol Screw_Terminal_01x05
- added K1, K2, K3: SANYOU_SRD_Form_C, Relays_THT:Relay_SPDT_SANYOU_SRD_Series_Form_C, symbol SANYOU_SRD_Form_C
- added R2, R3, R4: 10k, Resistors_SMD:R_0805_HandSoldering, symbol R
- added R5, R6: 300R, Resistors_SMD:R_0805_HandSoldering, symbol R
- added SW1: SW_Rotary8, windshield_wiper:ROT_SW_8, symbol SW_Rotary8
- C1, C3, C4: renamed from C?; footprint (none) -> Capacitors_SMD:C_0805_HandSoldering
- C2: renamed from C?; footprint (none) -> Capacitors_SMD:CP_Elec_6.3x5.3
- D2, D3, D4: renamed from D?; footprint (none) -> Diodes_SMD:D_SOD-123F
- J1: renamed from J?; footprint (none) -> Pin_Headers:Pin_Header_Straight_1x04_Pitch2.54mm
- Q1: renamed from Q?; footprint (none) -> TO_SOT_Packages_SMD:SOT-23_Handsoldering
- Q2, Q3, Q4: renamed from Q?; footprint (none) -> TO_SOT_Packages_SMD:SOT-323_SC-70_Handsoldering
- R1, R7, R8, R9: renamed from R?; footprint (none) -> Resistors_SMD:R_0805_HandSoldering
- U1: renamed from U?; footprint (none) -> TO_SOT_Packages_SMD:SOT-223-3_TabPin2
- U2: renamed from U?; footprint 20N -> Housings_DIP:DIP-20_W7.62mm_LongPads
Connections:
- net labels added: Fast, R1, R2, R3, SW_C, SW_NC, Slow
- wire segments 55 -> 140
- no-connect marks 0 -> 2
Other:
- note added: "2 position switch\n"
- note added: "On/Off button"
- note added: "Wiper Motor\n"
- moved on the sheet: Q2, Q3, Q4, R7, R8, R9
